File: Chibi-T_Furoshiki_AutoAirAdjust_PCB.kicad_pcb (KiCad board)
At the start: 2 copper layers, 50 x 50 mm, 40 parts, among them J1 M-BUS, J2 from_12V_Power, J3 from_5V_Power, J4 PRESSURE_SEN, J5 I2C, J6 I2C, J7 SOLENOID, Q1 AO3400A, U1 MP1584EN-LF-Z, U2 ADS1015IDGS

Commit message: docs: ソレノイドバルブ制御のGPIOを34から13に変更。Ver.1.00→1.01
Connections:
- net /GPIO18_1_1 renamed /GPIO18_1_1_1
- net /GPIO19_1_1 renamed /GPIO19_1_1_1
- net /GPIO1_1_1 renamed /GPIO1_1_1_1
- net /GPIO23_2_2 renamed /GPIO23_2_2_2
- net /GPIO25_2_2 renamed /GPIO25_2_2_2
- net /GPIO26_1_1 renamed /GPIO26_1_1_1
- net /GPIO2_1_1 renamed /GPIO2_1_1_1
- J1 pad 21: /GPIO13_1_1 -> SOL_TRG
- J1 pad 25: SOL_TRG -> /GPIO34_2
Routing:
- net SOL_TRG: track 50.6 -> 56.9 mm
- net /GPIO15: track 2.59 -> 0.00 mm
- net /GPIO0: track 1.86 -> 0.00 mm
Other:
- board text added: "Chibi-T Furoshiki AutoAirAdjust Ver.1.01 2026.07.14"
- board text removed: "Chibi-T Furoshiki AutoAirAdjust Ver.1.00 2026.07.11"
Changed lines of the file:
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@@
 	(paper "A4")
 	(title_block
-		(date "2026-07-12")
+		(date "2026-07-14")
+		(rev "1.01")
 	)
 	(layers
@@
 		(sheetname "/")
 		(sheetfile "Chibi-T_Furoshiki_AutoAirAdjust_PCB.kicad_sch")
+		(units
+			(unit
+				(name "A")
+				(pins "1" "2")
+			)
+		)
 		(attr through_hole)
 		(duplicate_pad_numbers_are_jumpers no)
@@
 			(size 1 1)
 			(layers "F.Cu" "F.Mask")
-			(net "/GPIO25_2_1")
+			(net "/GPIO25_2_2_1")
 			(pinfunction "Pin_7_7")
 			(pintype "passive+no_connect")
@@
 			(size 1 1)
 			(layers "B.Cu" "B.Mask")
-			(net "/GPIO25_2")
+			(net "/GPIO25_2_2")
 			(pinfunction "Pin_7_7")
 			(pintype "passive+no_connect")
@@
 			(layers "*.Cu" "*.Mask")
 			(remove_unused_layers no)
-			(net "/GPIO25_2_2")
+			(net "/GPIO25_2_2_2")
 			(pinfunction "Pin_7_7")
 			(pintype "passive+no_connect")
@@
 			(size 1 1)
 			(layers "F.Cu" "F.Mask")
-			(net "/GPIO23_2")
+			(net "/GPIO23_2_2")
 			(pinfunction "Pin_8_8")
 			(pintype "passive+no_connect")
@@
 			(size 1 1)
 			(layers "B.Cu" "B.Mask")
-			(net "/GPIO23_2_1")
+			(net "/GPIO23_2_2_1")
 			(pinfunction "Pin_8_8")
 			(pintype "passive+no_connect")
@@
 			(layers "*.Cu" "*.Mask")
 			(remove_unused_layers no)
-			(net "/GPIO23_2_2")
+			(net "/GPIO23_2_2_2")
 			(pinfunction "Pin_8_8")
 			(pintype "passive+no_connect")
@@
 			(size 1 1)
 			(layers "F.Cu" "F.Mask")
-			(net "/GPIO26_1_2")
+			(net "/GPIO26_1_1_2")
 			(pinfunction "Pin_9_9")
 			(pintype "passive+no_connect")
@@
 			(size 1 1)
 			(layers "B.Cu" "B.Mask")
-			(net "/GPIO26_1")
+			(net "/GPIO26_1_1")
 			(pinfunction "Pin_9_9")
 			(pintype "passive+no_connect")
@@
 			(layers "*.Cu" "*.Mask")
 			(remove_unused_layers no)
-			(net "/GPIO26_1_1")
+			(net "/GPIO26_1_1_1")
 			(pinfunction "Pin_9_9")
 			(pintype "passive+no_connect")
@@
 			(size 1 1)
 			(layers "F.Cu" "F.Mask")
-			(net "/GPIO19_1_2")
+			(net "/GPIO19_1_1_2")
 			(pinfunction "Pin_10_10")
 			(pintype "passive+no_connect")
@@
 			(size 1 1)
 			(layers "B.Cu" "B.Mask")
-			(net "/GPIO19_1")
+			(net "/GPIO19_1_1")
 			(pinfunction "Pin_10_10")
 			(pintype "passive+no_connect")
@@
 			(layers "*.Cu" "*.Mask")
 			(remove_unused_layers no)
-			(net "/GPIO19_1_1")
+			(net "/GPIO19_1_1_1")
 			(pinfunction "Pin_10_10")
 			(pintype "passive+no_connect")
@@
 			(size 1 1)
 			(layers "F.Cu" "F.Mask")
-			(net "/GPIO18_1")
+			(net "/GPIO18_1_1")
 			(pinfunction "Pin_12_12")
 			(pintype "passive+no_connect")
@@
 			(size 1 1)
 			(layers "B.Cu" "B.Mask")
-			(net "/GPIO18_1_2")
+			(net "/GPIO18_1_1_2")
 			(pinfunction "Pin_12_12")
 			(pintype "passive+no_connect")
@@
 			(layers "*.Cu" "*.Mask")
 			(remove_unused_layers no)
-			(net "/GPIO18_1_1")
+			(net "/GPIO18_1_1_1")
 			(pinfunction "Pin_12_12")
 			(pintype "passive+no_connect")
@@
 			(size 1 1)
 			(layers "F.Cu" "F.Mask")
-			(net "/GPIO1_1_2")
+			(net "/GPIO1_1_1_2")
 			(pinfunction "Pin_13_13")
 			(pintype "passive+no_connect")
@@
 			(size 1 1)
 			(layers "B.Cu" "B.Mask")
-			(net "/GPIO1_1")
+			(net "/GPIO1_1_1")
 			(pinfunction "Pin_13_13")
 			(pintype "passive+no_connect")
@@
 			(layers "*.Cu" "*.Mask")
 			(remove_unused_layers no)
-			(net "/GPIO1_1_1")
+			(net "/GPIO1_1_1_1")
 			(pinfunction "Pin_13_13")
 			(pintype "passive+no_connect")
@@
 			(net "/GPIO17")
 			(pinfunction "Pin_15_15")
-			(pintype "passive")
+			(pintype "passive+no_connect")
 			(zone_connect 0)
 			(options
@@
 			(net "/GPIO17")
 			(pinfunction "Pin_15_15")
-			(pintype "passive")
+			(pintype "passive+no_connect")
 			(zone_connect 0)
 			(options
@@
 			(net "/GPIO17")
 			(pinfunction "Pin_15_15")
-			(pintype "passive")
+			(pintype "passive+no_connect")
 		)
 		(pad "16" smd custom
@@
 			(net "/GPIO16")
 			(pinfunction "Pin_16_16")
-			(pintype "passive")
+			(pintype "passive+no_connect")
 			(zone_connect 0)
 			(options
@@
 			(net "/GPIO16")
 			(pinfunction "Pin_16_16")
-			(pintype "passive")
+			(pintype "passive+no_connect")
 			(zone_connect 0)
 			(options
@@
 			(net "/GPIO16")
 			(pinfunction "Pin_16_16")
-			(pintype "passive")
+			(pintype "passive+no_connect")
 		)
 		(pad "17" smd custom
@@
 			(size 1 1)
 			(layers "F.Cu" "F.Mask")
-			(net "/GPIO2_1_2")
+			(net "/GPIO2_1_1_2")
 			(pinfunction "Pin_20_20")
 			(pintype "passive+no_connect")
@@
 			(size 1 1)
 			(layers "B.Cu" "B.Mask")
-			(net "/GPIO2_1")
+			(net "/GPIO2_1_1")
 			(pinfunction "Pin_20_20")
 			(pintype "passive+no_connect")
@@
 			(layers "*.Cu" "*.Mask")
 			(remove_unused_layers no)
-			(net "/GPIO2_1_1")
+			(net "/GPIO2_1_1_1")
 			(pinfunction "Pin_20_20")
 			(pintype "passive+no_connect")
@@
 			(size 1 1)
 			(layers "F.Cu" "F.Mask")
-			(net "/GPIO13_1")
+			(net "SOL_TRG")
 			(pinfunction "Pin_21_21")
-			(pintype "passive+no_connect")
+			(pintype "passive")
 			(zone_connect 0)
 			(options
@@
 			(size 1 1)
 			(layers "B.Cu" "B.Mask")
-			(net "/GPIO13_1_2")
+			(net "SOL_TRG")
 			(pinfunction "Pin_21_21")
-			(pintype "passive+no_connect")
+			(pintype "passive")
 			(zone_connect 0)
 			(options
@@
 			(layers "*.Cu" "*.Mask")
 			(remove_unused_layers no)
-			(net "/GPIO13_1_1")
+			(net "SOL_TRG")
 			(pinfunction "Pin_21_21")
-			(pintype "passive+no_connect")
+			(pintype "passive")
 		)
 		(pad "22" smd custom
@@
 			(net "/GPIO0")
 			(pinfunction "Pin_23_23")
-			(pintype "passive")
+			(pintype "passive+no_connect")
 			(zone_connect 0)
 			(options
@@
 			(net "/GPIO0")
 			(pinfunction "Pin_23_23")
-			(pintype "passive")
+			(pintype "passive+no_connect")
 			(zone_connect 0)
 			(options
@@
 			(net "/GPIO0")
 			(pinfunction "Pin_23_23")
-			(pintype "passive")
+			(pintype "passive+no_connect")
 		)
 		(pad "24" smd custom
@@
 			(net "/GPIO15")
 			(pinfunction "Pin_24_24")
-			(pintype "passive")
+			(pintype "passive+no_connect")
 			(zone_connect 0)
 			(options
@@
 			(net "/GPIO15")
 			(pinfunction "Pin_24_24")
-			(pintype "passive")
+			(pintype "passive+no_connect")
 			(zone_connect 0)
 			(options
@@
 			(net "/GPIO15")
 			(pinfunction "Pin_24_24")
-			(pintype "passive")
+			(pintype "passive+no_connect")
 		)
 		(pad "25" smd custom
@@
 			(size 1 1)
 			(layers "F.Cu" "F.Mask")
-			(net "SOL_TRG")
+			(net "/GPIO34_2")
 			(pinfunction "Pin_25_25")
-			(pintype "passive")
+			(pintype "passive+no_connect")
 			(zone_connect 0)
 			(options
@@
 			(size 1 1)
 			(layers "B.Cu" "B.Mask")
-			(net "SOL_TRG")
+			(net "/GPIO34_2")
 			(pinfunction "Pin_25_25")
-			(pintype "passive")
+			(pintype "passive+no_connect")
 			(zone_connect 0)
 			(options
@@
 			(layers "*.Cu" "*.Mask")
 			(remove_unused_layers no)
-			(net "SOL_TRG")
+			(net "/GPIO34_2")
 			(pinfunction "Pin_25_25")
-			(pintype "passive")
+			(pintype "passive+no_connect")
 		)
 		(pad "26" smd custom
@@
 		)
 	)
-	(gr_text "Chibi-T Furoshiki\nAutoAirAdjust Ver.1.00  2026.07.11"
+	(gr_text "Chibi-T Furoshiki\nAutoAirAdjust Ver.1.01  2026.07.14"
 		(at 143.129 106.934 0)
 		(layer "B.SilkS")
@@
 	)
 	(segment
-		(start 110.376864 139.7)
-		(end 109.27 139.7)
+		(start 132.334 134.366)
+		(end 132.334 136.946194)
 		(width 0.6)
 		(layer "B.Cu")
@@
 	)
 	(segment
-		(start 132.334 136.946194)
-		(end 137.922 142.534194)
+		(start 117.7424 146.9524)
+		(end 114.3 143.51)
 		(width 0.6)
 		(layer "B.Cu")
@@
 	)
 	(segment
-		(start 137.922 144.78)
-		(end 135.7496 146.9524)
+		(start 134.239 132.461)
+		(end 132.334 134.366)
 		(width 0.6)
 		(layer "B.Cu")
@@
 	)
 	(segment
-		(start 135.7496 146.9524)
-		(end 117.629264 146.9524)
+		(start 137.922 142.534194)
+		(end 137.922 144.78)
 		(width 0.6)
 		(layer "B.Cu")
@@
 	)
 	(segment
-		(start 137.922 142.534194)
-		(end 137.922 144.78)
+		(start 137.922 144.78)
+		(end 135.7496 146.9524)
 		(width 0.6)
 		(layer "B.Cu")
@@
 	)
 	(segment
-		(start 134.239 132.461)
-		(end 132.334 134.366)
+		(start 114.3 136.398)
+		(end 112.522 134.62)
 		(width 0.6)
 		(layer "B.Cu")
@@
 	)
 	(segment
-		(start 132.334 134.366)
-		(end 132.334 136.946194)
+		(start 114.3 143.51)
+		(end 114.3 136.398)
 		(width 0.6)
 		(layer "B.Cu")
@@
 	)
 	(segment
-		(start 117.629264 146.9524)
-		(end 110.376864 139.7)
+		(start 135.7496 146.9524)
+		(end 117.7424 146.9524)
 		(width 0.6)
 		(layer "B.Cu")
@@
 	)
 	(segment
-		(start 111.126396 137.16)
-		(end 109.27 137.16)
-		(width 0.25)
-		(layer "F.Cu")
-		(net "/GPIO0")
+		(start 112.522 134.62)
+		(end 109.27 134.62)
+		(width 0.6)
+		(layer "B.Cu")
+		(net "SOL_TRG")
 	)
 	(segment
-		(start 106.73 137.16)
-		(end 104.14 137.16)
-		(width 0.4)
-		(layer "F.Cu")
-		(net "/GPIO15")
+		(start 132.334 136.946194)
+		(end 137.922 142.534194)
+		(width 0.6)
+		(layer "B.Cu")
+		(net "SOL_TRG")
 	)
 	(zone

Commit message: faeyure: I2CバスのGPIOピンを変更
Connections:
- net /GPIO0 renamed /GPIO0_2
- net /GPIO15 renamed /GPIO15_1
- net /GPIO16 renamed /GPIO16_2
- net /GPIO17 renamed /GPIO17_1
- net /GPIO18_1_1_1 renamed /GPIO18_1_1_1_1
- net /GPIO19_1_1_1 renamed /GPIO19_1_1_1_1
- net /GPIO1_1_1_1 renamed /GPIO1_1_1_1_1
- net /GPIO23_2_2_2 renamed /GPIO23_2_2_2_2
- net /GPIO25_2_2_2 renamed /GPIO25_2_2_2_2
- net /GPIO26_1_1_1 renamed /GPIO26_1_1_1_1
- net /GPIO34_2 renamed /GPIO34_2_2
- J1 pad 17: SCL -> /GPIO22_1
- J1 pad 18: SDA -> /GPIO21_2
- J1 pad 19: /GPIO5 -> SCL
- J1 pad 20: /GPIO2_1_1_1 -> SDA
Routing:
- net SDA: track 66.9 -> 64.3 mm
Other:
- board text added: "Chibi-T Furoshiki AutoAirAdjust Ver.1.02 2026.08.07"
- board text removed: "Chibi-T Furoshiki AutoAirAdjust Ver.1.01 2026.07.14"
Changed lines of the file:
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@@
 	(paper "A4")
 	(title_block
-		(date "2026-07-14")
-		(rev "1.01")
+		(date "2026-08-07")
+		(rev "1.02")
 	)
 	(layers
@@
 			(size 1 1)
 			(layers "F.Cu" "F.Mask")
-			(net "/GPIO25_2_2_1")
+			(net "/GPIO25_2_2_2_1")
 			(pinfunction "Pin_7_7")
 			(pintype "passive+no_connect")
@@
 			(size 1 1)
 			(layers "B.Cu" "B.Mask")
-			(net "/GPIO25_2_2")
+			(net "/GPIO25_2_2_2")
 			(pinfunction "Pin_7_7")
 			(pintype "passive+no_connect")
@@
 			(layers "*.Cu" "*.Mask")
 			(remove_unused_layers no)
-			(net "/GPIO25_2_2_2")
+			(net "/GPIO25_2_2_2_2")
 			(pinfunction "Pin_7_7")
 			(pintype "passive+no_connect")
@@
 			(size 1 1)
 			(layers "F.Cu" "F.Mask")
-			(net "/GPIO23_2_2")
+			(net "/GPIO23_2_2_2")
 			(pinfunction "Pin_8_8")
 			(pintype "passive+no_connect")
@@
 			(size 1 1)
 			(layers "B.Cu" "B.Mask")
-			(net "/GPIO23_2_2_1")
+			(net "/GPIO23_2_2_2_1")
 			(pinfunction "Pin_8_8")
 			(pintype "passive+no_connect")
@@
 			(layers "*.Cu" "*.Mask")
 			(remove_unused_layers no)
-			(net "/GPIO23_2_2_2")
+			(net "/GPIO23_2_2_2_2")
 			(pinfunction "Pin_8_8")
 			(pintype "passive+no_connect")
@@
 			(size 1 1)
 			(layers "F.Cu" "F.Mask")
-			(net "/GPIO26_1_1_2")
+			(net "/GPIO26_1_1_1_2")
 			(pinfunction "Pin_9_9")
 			(pintype "passive+no_connect")
@@
 			(size 1 1)
 			(layers "B.Cu" "B.Mask")
-			(net "/GPIO26_1_1")
+			(net "/GPIO26_1_1_1")
 			(pinfunction "Pin_9_9")
 			(pintype "passive+no_connect")
@@
 			(layers "*.Cu" "*.Mask")
 			(remove_unused_layers no)
-			(net "/GPIO26_1_1_1")
+			(net "/GPIO26_1_1_1_1")
 			(pinfunction "Pin_9_9")
 			(pintype "passive+no_connect")
@@
 			(size 1 1)
 			(layers "F.Cu" "F.Mask")
-			(net "/GPIO19_1_1_2")
+			(net "/GPIO19_1_1_1_2")
 			(pinfunction "Pin_10_10")
 			(pintype "passive+no_connect")
@@
 			(size 1 1)
 			(layers "B.Cu" "B.Mask")
-			(net "/GPIO19_1_1")
+			(net "/GPIO19_1_1_1")
 			(pinfunction "Pin_10_10")
 			(pintype "passive+no_connect")
@@
 			(layers "*.Cu" "*.Mask")
 			(remove_unused_layers no)
-			(net "/GPIO19_1_1_1")
+			(net "/GPIO19_1_1_1_1")
 			(pinfunction "Pin_10_10")
 			(pintype "passive+no_connect")
@@
 			(size 1 1)
 			(layers "F.Cu" "F.Mask")
-			(net "/GPIO18_1_1")
+			(net "/GPIO18_1_1_1")
 			(pinfunction "Pin_12_12")
 			(pintype "passive+no_connect")
@@
 			(size 1 1)
 			(layers "B.Cu" "B.Mask")
-			(net "/GPIO18_1_1_2")
+			(net "/GPIO18_1_1_1_2")
 			(pinfunction "Pin_12_12")
 			(pintype "passive+no_connect")
@@
 			(layers "*.Cu" "*.Mask")
 			(remove_unused_layers no)
-			(net "/GPIO18_1_1_1")
+			(net "/GPIO18_1_1_1_1")
 			(pinfunction "Pin_12_12")
 			(pintype "passive+no_connect")
@@
 			(size 1 1)
 			(layers "F.Cu" "F.Mask")
-			(net "/GPIO1_1_1_2")
+			(net "/GPIO1_1_1_1_2")
 			(pinfunction "Pin_13_13")
 			(pintype "passive+no_connect")
@@
 			(size 1 1)
 			(layers "B.Cu" "B.Mask")
-			(net "/GPIO1_1_1")
+			(net "/GPIO1_1_1_1")
 			(pinfunction "Pin_13_13")
 			(pintype "passive+no_connect")
@@
 			(layers "*.Cu" "*.Mask")
 			(remove_unused_layers no)
-			(net "/GPIO1_1_1_1")
+			(net "/GPIO1_1_1_1_1")
 			(pinfunction "Pin_13_13")
 			(pintype "passive+no_connect")
@@
 			(size 1 1)
 			(layers "F.Cu" "F.Mask")
-			(net "/GPIO17")
+			(net "/GPIO17_2")
 			(pinfunction "Pin_15_15")
 			(pintype "passive+no_connect")
@@
 			(layers "*.Cu" "*.Mask")
 			(remove_unused_layers no)
-			(net "/GPIO17")
+			(net "/GPIO17_1")
 			(pinfunction "Pin_15_15")
 			(pintype "passive+no_connect")
@@
 			(size 1 1)
 			(layers "F.Cu" "F.Mask")
-			(net "/GPIO16")
+			(net "/GPIO16_1")
 			(pinfunction "Pin_16_16")
 			(pintype "passive+no_connect")
@@
 			(layers "*.Cu" "*.Mask")
 			(remove_unused_layers no)
-			(net "/GPIO16")
+			(net "/GPIO16_2")
 			(pinfunction "Pin_16_16")
 			(pintype "passive+no_connect")
@@
 			(size 1 1)
 			(layers "F.Cu" "F.Mask")
-			(net "SCL")
+			(net "/GPIO22")
 			(pinfunction "Pin_17_17")
-			(pintype "passive")
+			(pintype "passive+no_connect")
 			(zone_connect 0)
 			(options
@@
 			(size 1 1)
 			(layers "B.Cu" "B.Mask")
-			(net "SCL")
+			(net "/GPIO22_2")
 			(pinfunction "Pin_17_17")
-			(pintype "passive")
+			(pintype "passive+no_connect")
 			(zone_connect 0)
 			(options
@@
 			(layers "*.Cu" "*.Mask")
 			(remove_unused_layers no)
-			(net "SCL")
+			(net "/GPIO22_1")
 			(pinfunction "Pin_17_17")
-			(pintype "passive")
+			(pintype "passive+no_connect")
 		)
 		(pad "18" smd custom
@@
 			(size 1 1)
 			(layers "F.Cu" "F.Mask")
-			(net "SDA")
+			(net "/GPIO21_1")
 			(pinfunction "Pin_18_18")
-			(pintype "passive")
+			(pintype "passive+no_connect")
 			(zone_connect 0)
 			(options
@@
 			(size 1 1)
 			(layers "B.Cu" "B.Mask")
-			(net "SDA")
+			(net "/GPIO21")
 			(pinfunction "Pin_18_18")
-			(pintype "passive")
+			(pintype "passive+no_connect")
 			(zone_connect 0)
 			(options
@@
 			(layers "*.Cu" "*.Mask")
 			(remove_unused_layers no)
-			(net "SDA")
+			(net "/GPIO21_2")
 			(pinfunction "Pin_18_18")
-			(pintype "passive")
+			(pintype "passive+no_connect")
 		)
 		(pad "19" smd custom
@@
 			(size 1 1)
 			(layers "F.Cu" "F.Mask")
-			(net "/GPIO5_2")
+			(net "SCL")
 			(pinfunction "Pin_19_19")
-			(pintype "passive+no_connect")
+			(pintype "passive")
 			(zone_connect 0)
 			(options
@@
 			(size 1 1)
 			(layers "B.Cu" "B.Mask")
-			(net "/GPIO5_1")
+			(net "SCL")
 			(pinfunction "Pin_19_19")
-			(pintype "passive+no_connect")
+			(pintype "passive")
 			(zone_connect 0)
 			(options
@@
 			(layers "*.Cu" "*.Mask")
 			(remove_unused_layers no)
-			(net "/GPIO5")
+			(net "SCL")
 			(pinfunction "Pin_19_19")
-			(pintype "passive+no_connect")
+			(pintype "passive")
 		)
 		(pad "20" smd custom
@@
 			(size 1 1)
 			(layers "F.Cu" "F.Mask")
-			(net "/GPIO2_1_1_2")
+			(net "SDA")
 			(pinfunction "Pin_20_20")
-			(pintype "passive+no_connect")
+			(pintype "passive")
 			(zone_connect 0)
 			(options
@@
 			(size 1 1)
 			(layers "B.Cu" "B.Mask")
-			(net "/GPIO2_1_1")
+			(net "SDA")
 			(pinfunction "Pin_20_20")
-			(pintype "passive+no_connect")
+			(pintype "passive")
 			(zone_connect 0)
 			(options
@@
 			(layers "*.Cu" "*.Mask")
 			(remove_unused_layers no)
-			(net "/GPIO2_1_1_1")
+			(net "SDA")
 			(pinfunction "Pin_20_20")
-			(pintype "passive+no_connect")
+			(pintype "passive")
 		)
 		(pad "21" smd custom
@@
 			(size 1 1)
 			(layers "F.Cu" "F.Mask")
-			(net "/GPIO0")
+			(net "/GPIO0_1")
 			(pinfunction "Pin_23_23")
 			(pintype "passive+no_connect")
@@
 			(layers "*.Cu" "*.Mask")
 			(remove_unused_layers no)
-			(net "/GPIO0")
+			(net "/GPIO0_2")
 			(pinfunction "Pin_23_23")
 			(pintype "passive+no_connect")
@@
 			(size 1 1)
 			(layers "F.Cu" "F.Mask")
-			(net "/GPIO15")
+			(net "/GPIO15_2")
 			(pinfunction "Pin_24_24")
 			(pintype "passive+no_connect")
@@
 			(layers "*.Cu" "*.Mask")
 			(remove_unused_layers no)
-			(net "/GPIO15")
+			(net "/GPIO15_1")
 			(pinfunction "Pin_24_24")
 			(pintype "passive+no_connect")
@@
 			(size 1 1)
 			(layers "B.Cu" "B.Mask")
-			(net "/GPIO34_2")
+			(net "/GPIO34_2_1")
 			(pinfunction "Pin_25_25")
 			(pintype "passive+no_connect")
@@
 			(layers "*.Cu" "*.Mask")
 			(remove_unused_layers no)
-			(net "/GPIO34_2")
+			(net "/GPIO34_2_2")
 			(pinfunction "Pin_25_25")
 			(pintype "passive+no_connect")
@@
 		)
 	)
-	(gr_text "Chibi-T Furoshiki\nAutoAirAdjust Ver.1.01  2026.07.14"
+	(gr_text "Chibi-T Furoshiki\nAutoAirAdjust Ver.1.02  2026.08.07"
 		(at 143.129 106.934 0)
 		(layer "B.SilkS")
@@
 	)
 	(segment
+		(start 112.775442 132.08)
+		(end 109.27 132.08)
+		(width 0.4)
+		(layer "B.Cu")
+		(net "SCL")
+	)
+	(segment
 		(start 124.61736 142.24)
 		(end 123.34748 143.50988)
@@
 	(segment
 		(start 123.34748 142.652038)
-		(end 110.235442 129.54)
+		(end 112.775442 132.08)
 		(width 0.4)
 		(layer "B.Cu")
@@
 	)
 	(segment
-		(start 108.0676 137.658051)
-		(end 108.0676 130.8776)
+		(start 121.34596 143.51)
+		(end 120.35856 144.4974)
 		(width 0.4)
 		(layer "F.Cu")
@@
 	)
 	(segment
-		(start 121.34596 143.51)
-		(end 120.35856 144.4974)
+		(start 108.0676 133.4176)
+		(end 106.73 132.08)
 		(width 0.4)
 		(layer "F.Cu")
@@
 	)
 	(segment
-		(start 108.771949 138.3624)
-		(end 108.0676 137.658051)
+		(start 108.0676 137.658051)
+		(end 108.0676 133.4176)
 		(width 0.4)
 		(layer "F.Cu")
@@
 	)
 	(segment
-		(start 108.0676 130.8776)
-		(end 106.73 129.54)
+		(start 108.771949 138.3624)
+		(end 108.0676 137.658051)
 		(width 0.4)
 		(layer "F.Cu")
