File: Chibi-T_Furoshiki_AutoAirAdjust_PCB.kicad_sch (KiCad schematic)
At the start: 39 parts, among them J1 M-BUS, J2 from_12V_Power, J3 from_5V_Power, J4 PRESSURE_SEN, J5 I2C, J6 I2C, J7 SOLENOID, Q1 AO3400A, U1 MP1584EN-LF-Z, U2 ADS1015IDGS

Commit message: docs: ソレノイドバルブ制御のGPIOを34から13に変更。Ver.1.00→1.01
Connections:
- net GPIO13_1_1 is gone; now on net SOL_TRG: J1.21 (Pin_21)
- net SOL_TRG: no longer J1.25 (Pin_25)
- net GPIO18_1_1 renamed GPIO18_1_1_1
- net GPIO19_1_1 renamed GPIO19_1_1_1
- net GPIO1_1_1 renamed GPIO1_1_1_1
- net GPIO23_2_2 renamed GPIO23_2_2_2
- net GPIO25_2_2 renamed GPIO25_2_2_2
- net GPIO26_1_1 renamed GPIO26_1_1_1
- net GPIO2_1_1 renamed GPIO2_1_1_1
- new net GPIO34_2: J1.25 (Pin_25)
- no-connect marks 15 -> 19
Changed lines of the file:
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@@
 	(paper "A4")
 	(title_block
-		(date "2022-10-23")
+		(date "2026-07-14")
+		(rev "1.01")
 	)
 	(text "Core1"
@@
 	)
 	(no_connect
+		(at 110.49 113.03)
+	)
+	(no_connect
 		(at 123.19 107.95)
 	)
@@
 	)
 	(no_connect
+		(at 123.19 113.03)
+	)
+	(no_connect
 		(at 123.19 90.17)
 	)
@@
 	)
 	(no_connect
+		(at 123.19 115.57)
+	)
+	(no_connect
 		(at 123.19 100.33)
 	)
@@
 	)
 	(no_connect
-		(at 123.19 110.49)
+		(at 110.49 102.87)
 	)
 	(no_connect
@@
 	)
 	(no_connect
+		(at 123.19 102.87)
+	)
+	(no_connect
 		(at 123.19 92.71)
 	)
@@
 	(wire
 		(pts
-			(xy 123.19 115.57) (xy 139.7 115.57)
-		)
-		(stroke
-			(width 0)
-			(type default)
-		)
-	)
-	(wire
-		(pts
 			(xy 99.06 43.18) (xy 101.6 43.18)
 		)
@@
 	(wire
 		(pts
+			(xy 123.19 110.49) (xy 139.7 110.49)
+		)
+		(stroke
+			(width 0)
+			(type default)
+		)
+	)
+	(wire
+		(pts
 			(xy 78.74 83.82) (xy 78.74 85.09)
 		)
@@
 		)
 	)
-	(label "GPIO19_1_1"
+	(label "GPIO19_1_1_1"
 		(at 110.49 95.25 180)
 		(effects
@@
 		)
 	)
-	(label "GPIO18_1_1"
+	(label "GPIO18_1_1_1"
 		(at 110.49 97.79 180)
 		(effects
@@
 		)
 	)
-	(label "GPIO26_1_1"
+	(label "GPIO26_1_1_1"
 		(at 123.19 95.25 0)
 		(effects
@@
 		)
 	)
-	(label "GPIO1_1_1"
+	(label "GPIO1_1_1_1"
 		(at 123.19 100.33 0)
 		(effects
@@
 		)
 	)
-	(label "GPIO25_2_2"
+	(label "GPIO25_2_2_2"
 		(at 123.19 92.71 0)
 		(effects
@@
 		)
 	)
-	(label "GPIO23_2_2"
+	(label "GPIO23_2_2_2"
 		(at 110.49 92.71 180)
 		(effects
@@
 		)
 	)
-	(label "GPIO2_1_1"
+	(label "GPIO2_1_1_1"
 		(at 110.49 107.95 180)
 		(effects
@@
 		)
 	)
-	(global_label "SOL_TRG"
-		(shape output)
-		(at 139.7 115.57 0)
-		(fields_autoplaced yes)
-		(effects
-			(font
-				(size 1.27 1.27)
-			)
-			(justify left)
-		)
-		(property "Intersheetrefs" "${INTERSHEET_REFS}"
-			(at 150.7285 115.57 0)
-			(hide yes)
-			(show_name no)
-			(do_not_autoplace no)
-			(effects
-				(font
-					(size 1.27 1.27)
-				)
-				(justify left)
-			)
-		)
-	)
 	(global_label "AIN0"
 		(shape output)
@@
 			)
 		)
+	)
+	(global_label "SOL_TRG"
+		(shape output)
+		(at 139.7 110.49 0)
+		(fields_autoplaced yes)
+		(effects
+			(font
+				(size 1.27 1.27)
+			)
+			(justify left)
+		)
+		(property "Intersheetrefs" "${INTERSHEET_REFS}"
+			(at 150.7285 110.49 0)
+			(hide yes)
+			(show_name no)
+			(do_not_autoplace no)
+			(effects
+				(font
+					(size 1.27 1.27)
+				)
+				(justify left)
+			)
+		)

Commit message: faeyure: I2CバスのGPIOピンを変更
Connections:
- net GPIO2_1_1_1 is gone; now on net SDA: J1.20 (Pin_20)
- net GPIO5 is gone; now on net SCL: J1.19 (Pin_19)
- net SCL: no longer J1.17 (Pin_17)
- net SDA: no longer J1.18 (Pin_18)
- new net GPIO21: J1.18 (Pin_18)
- new net GPIO22: J1.17 (Pin_17)
Changed lines of the file:
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@@
 	(paper "A4")
 	(title_block
-		(date "2026-07-14")
-		(rev "1.01")
+		(date "2026-08-07")
+		(rev "1.02")
 	)
 	(text "Core1"
@@
 	)
 	(no_connect
-		(at 110.49 107.95)
-	)
-	(no_connect
 		(at 110.49 97.79)
 	)
@@
 	)
 	(no_connect
-		(at 123.19 107.95)
-	)
-	(no_connect
 		(at 110.49 110.49)
 	)
@@
 	)
 	(no_connect
+		(at 123.19 105.41)
+	)
+	(no_connect
+		(at 110.49 105.41)
+	)
+	(no_connect
 		(at 110.49 102.87)
 	)
@@
 	(wire
 		(pts
-			(xy 123.19 105.41) (xy 139.7 105.41)
-		)
-		(stroke
-			(width 0)
-			(type default)
-		)
-	)
-	(wire
-		(pts
 			(xy 153.67 38.1) (xy 153.67 41.91)
 		)
@@
 	(wire
 		(pts
-			(xy 93.98 105.41) (xy 110.49 105.41)
-		)
-		(stroke
-			(width 0)
-			(type default)
-		)
-	)
-	(wire
-		(pts
 			(xy 74.93 154.94) (xy 85.09 154.94)
 		)
@@
 	(wire
 		(pts
+			(xy 93.98 107.95) (xy 110.49 107.95)
+		)
+		(stroke
+			(width 0)
+			(type default)
+		)
+	)
+	(wire
+		(pts
 			(xy 78.74 115.57) (xy 110.49 115.57)
 		)
@@
 	(wire
 		(pts
+			(xy 123.19 107.95) (xy 139.7 107.95)
+		)
+		(stroke
+			(width 0)
+			(type default)
+		)
+	)
+	(wire
+		(pts
 			(xy 93.98 172.72) (xy 100.33 172.72)
 		)
@@
 	(global_label "SDA"
 		(shape input)
-		(at 93.98 105.41 180)
+		(at 93.98 107.95 180)
 		(fields_autoplaced yes)
 		(effects
@@
 		)
 		(property "Intersheetrefs" "${INTERSHEET_REFS}"
-			(at 87.4267 105.41 0)
+			(at 87.4267 107.95 0)
 			(hide yes)
 			(show_name no)
@@
 	(global_label "SCL"
 		(shape output)
-		(at 139.7 105.41 0)
+		(at 139.7 107.95 0)
 		(fields_autoplaced yes)
 		(effects
@@
 		)
 		(property "Intersheetrefs" "${INTERSHEET_REFS}"
-			(at 146.1928 105.41 0)
+			(at 146.1928 107.95 0)
 			(hide yes)
 			(show_name no)

Commit message: feature: 燃圧センサの断線検知用プルダウン抵抗を追加
Parts:
- added R10: 100k, Resistor_SMD:R_0603_1608Metric, symbol Device:R
Connections:
- net AIN0: now also R10.1
- net GND: now also R10.2
Changed lines of the file:
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@@
 	(paper "A4")
 	(title_block
-		(date "2026-08-07")
-		(rev "1.02")
+		(date "2026-08-16")
+		(rev "1.03")
 	)
 	(text "Core1"
@@
 	)
 	(junction
+		(at 26.67 167.64)
+		(diameter 0)
+		(color 0 0 0 0)
+	)
+	(junction
 		(at 132.08 38.1)
 		(diameter 0)
@@
 	)
 	(junction
+		(at 35.56 182.88)
+		(diameter 0)
+		(color 0 0 0 0)
+	)
+	(junction
 		(at 86.36 64.77)
 		(diameter 0)
@@
 	(wire
 		(pts
+			(xy 26.67 167.64) (xy 26.67 171.45)
+		)
+		(stroke
+			(width 0)
+			(type default)
+		)
+	)
+	(wire
+		(pts
 			(xy 35.56 182.88) (xy 55.88 182.88)
 		)
@@
 	(wire
 		(pts
+			(xy 26.67 182.88) (xy 26.67 179.07)
+		)
+		(stroke
+			(width 0)
+			(type default)
+		)
+	)
+	(wire
+		(pts
 			(xy 85.09 158.75) (xy 85.09 154.94)
 		)
@@
 	(wire
 		(pts
+			(xy 22.86 167.64) (xy 26.67 167.64)
+		)
+		(stroke
+			(width 0)
+			(type default)
+		)
+	)
+	(wire
+		(pts
 			(xy 107.95 40.64) (xy 107.95 46.99)
 		)
@@
 	(wire
 		(pts
+			(xy 35.56 182.88) (xy 26.67 182.88)
+		)
+		(stroke
+			(width 0)
+			(type default)
+		)
+	)
+	(wire
+		(pts
 			(xy 38.1 114.3) (xy 38.1 115.57)
 		)
@@
 	(wire
 		(pts
+			(xy 26.67 167.64) (xy 45.72 167.64)
+		)
+		(stroke
+			(width 0)
+			(type default)
+		)
+	)
+	(wire
+		(pts
 			(xy 160.02 114.3) (xy 160.02 120.65)
 		)
@@
 	(wire
 		(pts
-			(xy 27.94 167.64) (xy 45.72 167.64)
-		)
-		(stroke
-			(width 0)
-			(type default)
-		)
-	)
-	(wire
-		(pts
 			(xy 38.1 115.57) (xy 49.53 115.57)
 		)
@@
 	(global_label "AIN0"
 		(shape input)
-		(at 27.94 167.64 180)
+		(at 22.86 167.64 180)
 		(fields_autoplaced yes)
 		(effects
@@
 		)
 		(property "Intersheetrefs" "${INTERSHEET_REFS}"
-			(at 20.7214 167.64 0)
+			(at 15.6414 167.64 0)
 			(hide yes)
 			(show_name no)
@@
 					(unit 1)
 				)
+			)
+		)
+	)
+	(symbol
+		(lib_id "Device:R")
+		(at 26.67 175.26 0)
+		(unit 1)
+		(body_style 1)
+		(exclude_from_sim no)
+		(in_bom yes)
+		(on_board yes)
+		(in_pos_files yes)
+		(dnp no)
+		(fields_autoplaced yes)
+		(property "Reference" "R10"
+			(at 29.21 173.9899 0)
+			(show_name no)
+			(do_not_autoplace no)
+			(effects
+				(font
+					(size 1.27 1.27)
+				)
+				(justify left)
+			)
+		)
+		(property "Value" "100k"
+			(at 29.21 176.5299 0)
+			(show_name no)
+			(do_not_autoplace no)
+			(effects
+				(font
+					(size 1.27 1.27)
+				)
+				(justify left)
+			)
+		)
+		(property "Footprint" "Resistor_SMD:R_0603_1608Metric"
+			(at 24.892 175.26 90)
+			(hide yes)
+			(show_name no)
+			(do_not_autoplace no)
+			(effects
+				(font
+					(size 1.27 1.27)
+				)
+			)
+		)
+		(property "Datasheet" ""
+			(at 26.67 175.26 0)
+			(hide yes)
+			(show_name no)
+			(do_not_autoplace no)
+			(effects
+				(font
+					(size 1.27 1.27)
+				)
+			)
+		)
+		(property "Description" "Resistor - AIN0 sensor disconnect pull-down (JST-XH J4 pin2 open-wire detect)"
+			(at 26.67 175.26 0)
+			(hide yes)
+			(show_name no)
+			(do_not_autoplace no)
+			(effects
+				(font
+					(size 1.27 1.27)
+				)
+			)
+		)
+		(property "LCSC" "C25803"
+			(at 26.67 175.26 0)
+			(hide yes)
+			(show_name no)
+			(do_not_autoplace no)
+			(effects
+				(font
+					(size 1.27 1.27)
+				)
+			)
+		)
+		(property "KiLib_Generator" "SMD_2terminal_chip_molded"
+			(at 26.67 175.26 0)
+			(hide yes)
+			(show_name no)
+			(do_not_autoplace no)
+			(effects
+				(font
+					(size 1.27 1.27)
+				)
+			)
+		)
+		(pin "1"
+		)
+		(pin "2"
+		)
+		(instances
+			(project "Chibi-T_Furoshiki_AutoAirAdjust_PCB"
+				(path "/70c425e8-c82b-42c0-a373-0ea779731c61"
+					(reference "R10")
+					(unit 1)
+				)
